Commit message: Use meshes for visual geometry

File: urdf/box_bot_geometric.urdf (robot description, URDF)
Before this commit: robot my_box_bot, 10 links, 9 joints
Links:
- link chassis: geometry visual mesh filename=package://my_box_bot_description/meshes/cute_cube.dae scale=0.1 0.1 0.1

Commit message: Solution

File: urdf/box_bot_geometric.urdf (robot description, URDF)
Before this commit: robot my_box_bot, 10 links, 9 joints
Joints:
- joint back_pitch_joint: axis (none) -> 0 1 0; limit (none) -> effort=1000.0 velocity=100.0
- joint back_roll_joint: axis (none) -> 1 0 0; limit (none) -> effort=1000.0 velocity=100.0
- joint back_yaw_joint: axis (none) -> 0 0 1; limit (none) -> effort=1000.0 velocity=100.0
- joint front_pitch_joint: axis (none) -> 0 1 0; limit (none) -> effort=1000.0 velocity=100.0
- joint front_roll_joint: axis (none) -> 1 0 0; limit (none) -> effort=1000.0 velocity=100.0
- joint front_yaw_joint: axis (none) -> 0 0 1; limit (none) -> effort=1000.0 velocity=100.0
- joint joint_left_wheel: axis (none) -> 0 1 0; limit (none) -> effort=10000 velocity=1000
- joint joint_right_wheel: axis (none) -> 0 1 0; limit (none) -> effort=10000 velocity=1000
